File: pitchfork_205_lqfp100.sch (KiCad schematic (older format))
At the start: 82 parts, among them P1 SD_CARD, P7 USB-MINI-B, SW1 SW_PUSH, SW2 SW_PUSH, SW3 SW_PUSH, SW4 SW_PUSH, U1 STM32F205Vxx, U2 NRF24L01+, U3 MCP73833, U6 LP38691, X1 CRYSTAL, X2 3.2x2.5, Y1 CHIP_ANTENNA

Commit message: [enh] 1st review, traces drawn
Parts:
- removed B1: SWITCH_4PIN, symbol SWITCH_4PIN
- removed C1, C2: 2.2u, symbol C
- removed C10, C11, C12, C13, C14, C8, C9: 100n, symbol CSMALL
- removed P7: USB-MINI-B, ~, symbol USB-MINI-B
- removed R10, R12, R8: 47k, ~, symbol R
- removed R11, R5, R7, R9: 1k, ~, symbol R
- removed R15: 2.2k, ~, symbol R
- removed R16: R, ~, symbol R
- removed R17: 150k, ~, symbol R
- removed U3: MCP73833, symbol MCP73833_CRIPPLED
- removed U6: LP38691, symbol LP38691
- added BT1: BATTERY_LI-ION, ~, symbol BATTERY_LI-ION
- added C1: 4.7uF, ~, symbol CSMALL
- added C2: 10uF, ~, symbol CSMALL
- added C41, C43: 2.2uF, ~, symbol CSMALL
- added C42: 0.1uF, ~, symbol CSMALL
- added L7: 10uH, ~, symbol INDUCTOR_SMALL
- added R7: 560k, symbol R_MINI
- added SW5: SWITCH_PUSHBUTTON, ~, symbol SWITCH_PUSHBUTTON
- added U3: USBCONN, symbol USBCONN
- added U4: LM3670, ~, symbol LM3670
- added U5: MCP73832-2, ~, symbol MCP73831/2
- added U6: UG-2864H, symbol UG-2864H
- C22: value 100n -> 10uF; footprint (none) -> ~
- C39: value 10uF -> 2.2uF
- C40: value 10uF -> 0.1uF
- R6: value 47k -> 2k
Connections:
- net labels added: +3.7V, BAT_CHRG, lcd_cs, lcd_d0, lcd_d1, lcd_d2, lcd_d3, lcd_d4, lcd_d5, lcd_d6, lcd_d7, lcd_rd, lcd_res, lcd_w, pa10, pb13, pb14, pb15, pc1, pd12, pd13
- net labels removed: VBAT, X1_1, X1_2, X1_3, pa0, pa1, pa2, pa3, pb0, pb1, pb2, pd0, pd1, pd4, pd5, pd7, pe10, pe6, pe7, pe8, pe9, usb_id, user_led, vbat
- wire segments 288 -> 299
Other:
- note added: "LCD"
- moved on the sheet: D1, D2, D3, D4, JP2, L1, L2, R1, R13, R14, R2, R4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
