File: small/pitchfork_205_lqfp64.sch (KiCad schematic (older format))
At the start: 78 parts, among them IC1 STM32F2XX_64LQFP, K1 CONN_3, P2 CONN_1, P3 CONN_1, SW1 EP11S1D1SAPE, SW2 EP11S1D1SAPE, SW3 EP11S1D1SAPE, SW4 EP11S1D1SAPE, SW5 EP11S1D1SAPE, U1 LM3670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

Commit message: [mod] update after kicad upgrade of baseboard
Parts:
- D1: symbol LED -> LED-RESCUE-pitchfork_205_lqfp64
- L2: symbol INDUCTOR -> INDUCTOR-RESCUE-pitchfork_205_lqfp64
Changed lines of the file:
@@
 $EndComp
 $Comp
-L INDUCTOR L2
+L INDUCTOR-RESCUE-pitchfork_205_lqfp64 L2
 U 1 1 51E3A64F
 P 2450 3300
@@
 $EndComp
 $Comp
-L LED D1
+L LED-RESCUE-pitchfork_205_lqfp64 D1
 U 1 1 533F38A2
 P 9400 3350
@@
 	10050 2350 10250 2350
 Wire Wire Line
-	10250 2350 10250 2500
-Wire Wire Line
-	9000 3350 9200 3350
+	10250 2350 10250 2600
+Wire Wire Line
+	8900 3350 9200 3350
 Wire Wire Line
 	3550 2800 3400 2800

Commit message: [fix] bugs from 2nd revision fixed
Parts:
- removed P2, P3: CONN_1, pitchfork:solderpad, symbol CONN_1
- added C36: 4.7uF, opendous:SM0603_Opendous, symbol C_Small
- added R12: 10k, opendous:0603_Opendous, symbol R
- SW_RFPWR1: value GS02MSABE -> EG1257; symbol SPST -> SW_SPDT
- U8: footprint DFN/QFN:DFN-8-1EP_2x2mm_Pitch0.5mm -> pitchforkv02:DFN-8-1EP_2x2mm_Pitch0.5mm
Connections:
- net labels removed: spare2, spare3
- wire segments 269 -> 273
Changed lines of the file:
@@
 LCD_RES
 $Comp
-L SPST SW_RFPWR1
+L SW_SPDT SW_RFPWR1
 U 1 1 543545A2
 P 8000 3350
-F 0 "SW_RFPWR1" H 8000 3450 70  0000 C CNN
-F 1 "GS02MSABE" H 8000 3250 70  0001 C CNN
+F 0 "SW_RFPWR1" H 8050 3550 70  0000 C CNN
+F 1 "EG1257" H 8000 3250 70  0001 C CNN
 F 2 "pitchforkbuttons:EG1257" H 8000 3350 60  0001 C CNN
 F 3 "~" H 8000 3350 60  0000 C CNN
@@
 Text Label 5550 4450 0    20   ~ 0
 btn3
-Text Label 5550 5200 0    20   ~ 0
-spare2
-Text Label 5550 5300 0    20   ~ 0
-spare3
-$Comp
-L CONN_1 P2
-U 1 1 5548EC51
-P 5850 5200
-F 0 "P2" H 5930 5200 40  0000 L CNN
-F 1 "CONN_1" H 5850 5255 30  0001 C CNN
-F 2 "pitchfork:solderpad" H 5850 5200 60  0001 C CNN
-F 3 "" H 5850 5200 60  0000 C CNN
-	1    5850 5200
-	1    0    0    -1
-$EndComp
-$Comp
-L CONN_1 P3
-U 1 1 5548EC57
-P 5850 5300
-F 0 "P3" H 5930 5300 40  0000 L CNN
-F 1 "CONN_1" H 5850 5355 30  0001 C CNN
-F 2 "pitchfork:solderpad" H 5850 5300 60  0001 C CNN
-F 3 "" H 5850 5300 60  0000 C CNN
-	1    5850 5300
-	1    0    0    -1
-$EndComp
 $Comp
 L GND #PWR031
@@
 F 0 "U8" H 8200 4700 50  0000 L CNN
 F 1 "TSV912" H 8200 4400 39  0000 L CNN
-F 2 "DFN/QFN:DFN-8-1EP_2x2mm_Pitch0.5mm" H 8100 4600 50  0001 C CNN
+F 2 "pitchforkv02:DFN-8-1EP_2x2mm_Pitch0.5mm" H 8100 4600 50  0001 C CNN
 F 3 "" H 8200 4700 50  0000 C CNN
 	1    8200 4550
@@
 F 0 "U8" H 9100 4700 50  0000 L CNN
 F 1 "TSV912" H 9100 4400 39  0000 L CNN
-F 2 "DFN/QFN:DFN-8-1EP_2x2mm_Pitch0.5mm" H 9000 4600 50  0001 C CNN
+F 2 "pitchforkv02:DFN-8-1EP_2x2mm_Pitch0.5mm" H 9000 4600 50  0001 C CNN
 F 3 "" H 9100 4700 50  0000 C CNN
 	2    9100 4550
@@
 	6350 2300 6350 2350
 Wire Wire Line
-	7450 3350 7500 3350
+	7450 3350 7800 3350
 Wire Wire Line
 	5700 6950 5500 6950
@@
 	10350 1850 10700 1850
 Wire Wire Line
-	8000 2750 8750 2750
+	7750 2750 8750 2750
 Wire Wire Line
 	8500 2550 8500 3350
@@
 Wire Wire Line
 	5500 4450 5700 4450
-Wire Wire Line
-	5500 5200 5700 5200
-Wire Wire Line
-	5500 5300 5700 5300
 Wire Wire Line
 	5500 4600 5900 4600
@@
 RNG
 Wire Wire Line
-	8500 3350 8600 3350
+	8200 3350 8600 3350
 Wire Wire Line
 	6800 1600 6700 1600
@@
 Wire Wire Line
 	3400 2800 3400 2850
+Wire Wire Line
+	8200 3250 8200 3350
+Wire Wire Line
+	8200 3450 8200 3500
+Wire Wire Line
+	8200 3500 8350 3500
+$Comp
+L R R12
+U 1 1 58E52A88
+P 8500 3500
+F 0 "R12" V 8580 3500 50  0000 C CNN
+F 1 "10k" V 8500 3500 50  0000 C CNN
+F 2 "opendous:0603_Opendous" V 8430 3500 50  0001 C CNN
+F 3 "" H 8500 3500 50  0000 C CNN
+	1    8500 3500
+	0    1    1    0
+$EndComp
+$Comp
+L GND #PWR041
+U 1 1 58E52BA6
+P 8750 3500
+F 0 "#PWR041" H 8750 3250 50  0001 C CNN
+F 1 "GND" H 8750 3350 50  0000 C CNN
+F 2 "" H 8750 3500 50  0000 C CNN
+F 3 "" H 8750 3500 50  0000 C CNN
+	1    8750 3500
+	1    0    0    -1
+$EndComp
+Wire Wire Line
+	8650 3500 8750 3500
+$Comp
+L GND #PWR042
+U 1 1 58E5441F
+P 850 1900
+F 0 "#PWR042" H 850 1650 50  0001 C CNN
+F 1 "GND" H 850 1750 50  0000 C CNN
+F 2 "" H 850 1900 50  0000 C CNN
+F 3 "" H 850 1900 50  0000 C CNN
+	1    850  1900
+	1    0    0    -1
+$EndComp
+Wire Wire Line
+	1050 1850 850  1850
+Wire Wire Line
+	850  1850 850  1900
+Connection ~ 8000 2750
+$Comp
+L C_Small C36
+U 1 1 58E551D9
+P 7750 2850
+F 0 "C36" H 7760 2920 30  0000 L CNN
+F 1 "4.7uF" H 7760 2770 30  0000 L CNN
+F 2 "opendous:SM0603_Opendous" H 7750 2850 50  0001 C CNN
+F 3 "" H 7750 2850 50  0000 C CNN
+	1    7750 2850
+	1    0    0    -1
+$EndComp
+$Comp
+L GND #PWR043
+U 1 1 58E5529C
+P 7750 2950
+F 0 "#PWR043" H 7750 2700 50  0001 C CNN
+F 1 "GND" H 7750 2800 50  0001 C CNN
+F 2 "" H 7750 2950 50  0000 C CNN
+F 3 "" H 7750 2950 50  0000 C CNN
+	1    7750 2950
+	1    0    0    -1
+$EndComp
 $EndSCHEMATC
