File: nokia/pitchfork_205_lqfp64.sch (KiCad schematic (older format))
At the start: 72 parts, among them IC1 STM32F2XX_64LQFP, K1 CONN_3, U1 LM3670, U2 USBCONN, U3 MCP73832-2, U4 NRF24L01+, U5 MC74VHC1G66, U6 MICROSDCARD, U7 TSV912, U8 TC75W57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

Commit message: [fix] lcd pinout + added R for nrf switch
Parts:
- removed D1: SML-211YTT86, opendous:0805_Opendous, symbol LED-RESCUE-pitchfork_205_lqfp64
- removed R2: 1k, opendous:0603_Opendous, symbol R
- added R11: 10k, opendous:0603_Opendous, symbol R_Small
- B1: symbol 3310 -> 3310-RESCUE-pitchfork_205_lqfp64
- SW_RFPWR1: value GS02MSABE -> EG1257; symbol SPST -> SW_DPDT_x2
Changed lines of the file:
@@
 usb_5v
-$Comp
-L GND #PWR019
-U 1 1 533F3896
-P 9850 3450
-F 0 "#PWR019" H 9850 3450 30  0001 C CNN
-F 1 "GND" H 9850 3380 30  0001 C CNN
-F 2 "" H 9850 3450 60  0001 C CNN
-F 3 "" H 9850 3450 60  0001 C CNN
-	1    9850 3450
-	1    0    0    -1
-$EndComp
-$Comp
-L R R2
-U 1 1 533F389C
-P 8750 3350
-F 0 "R2" V 8830 3350 50  0000 C CNN
-F 1 "1k" V 8750 3350 50  0000 C CNN
-F 2 "opendous:0603_Opendous" H 8750 3350 60  0001 C CNN
-F 3 "" H 8750 3350 60  0001 C CNN
-	1    8750 3350
-	0    -1   -1   0
-$EndComp
-$Comp
-L LED-RESCUE-pitchfork_205_lqfp64 D1
-U 1 1 533F38A2
-P 9400 3350
-F 0 "D1" H 9400 3450 50  0000 C CNN
-F 1 "SML-211YTT86" H 9400 3250 50  0000 C CNN
-F 2 "opendous:0805_Opendous" H 9400 3350 60  0001 C CNN
-F 3 "" H 9400 3350 60  0001 C CNN
-	1    9400 3350
-	1    0    0    -1
-$EndComp
 $Comp
 L STM32F2XX_64LQFP IC1
@@
 $EndComp
 $Comp
-L GND #PWR020
+L GND #PWR019
 U 1 1 53BDCC52
 P 3400 7550
-F 0 "#PWR020" H 3400 7550 30  0001 C CNN
+F 0 "#PWR019" H 3400 7550 30  0001 C CNN
 F 1 "GND" H 3400 7480 30  0001 C CNN
 F 2 "" H 3400 7550 60  0000 C CNN
@@
 $EndComp
 $Comp
-L GND #PWR021
+L GND #PWR020
 U 1 1 53BDE1E8
 P 4000 7250
-F 0 "#PWR021" H 4000 7250 30  0001 C CNN
+F 0 "#PWR020" H 4000 7250 30  0001 C CNN
 F 1 "GND" H 4000 7180 30  0001 C CNN
 F 2 "" H 4000 7250 60  0000 C CNN
@@
 $EndComp
 $Comp
-L GND #PWR022
+L GND #PWR021
 U 1 1 53BDE1F7
 P 4200 7250
-F 0 "#PWR022" H 4200 7250 30  0001 C CNN
+F 0 "#PWR021" H 4200 7250 30  0001 C CNN
 F 1 "GND" H 4200 7180 30  0001 C CNN
 F 2 "" H 4200 7250 60  0000 C CNN
@@
 $EndComp
 $Comp
-L GND #PWR023
+L GND #PWR022
 U 1 1 53BDE206
 P 4400 7250
-F 0 "#PWR023" H 4400 7250 30  0001 C CNN
+F 0 "#PWR022" H 4400 7250 30  0001 C CNN
 F 1 "GND" H 4400 7180 30  0001 C CNN
 F 2 "" H 4400 7250 60  0000 C CNN
@@
 LCD_RES
 $Comp
-L SPST SW_RFPWR1
+L SW_DPDT_x2 SW_RFPWR1
 U 1 1 543545A2
 P 8000 3350
-F 0 "SW_RFPWR1" H 8000 3450 70  0000 C CNN
-F 1 "GS02MSABE" H 8000 3250 70  0000 C CNN
+F 0 "SW_RFPWR1" H 8000 3550 70  0001 C CNN
+F 1 "EG1257" H 8000 3250 70  0001 C CNN
 F 2 "pitchforkbuttons:EG1257" H 8000 3350 60  0001 C CNN
 F 3 "~" H 8000 3350 60  0000 C CNN
@@
 $EndComp
 $Comp
-L GND #PWR024
+L GND #PWR023
 U 1 1 54C3B1D6
 P 6050 1150
-F 0 "#PWR024" H 6050 1150 30  0001 C CNN
+F 0 "#PWR023" H 6050 1150 30  0001 C CNN
 F 1 "GND" H 6050 1080 30  0001 C CNN
 F 2 "" H 6050 1150 60  0000 C CNN
@@
 $EndComp
 $Comp
-L GND #PWR025
+L GND #PWR024
 U 1 1 54C3C3E1
 P 8250 2950
-F 0 "#PWR025" H 8250 2950 30  0001 C CNN
+F 0 "#PWR024" H 8250 2950 30  0001 C CNN
 F 1 "GND" H 8250 2880 30  0001 C CNN
 F 2 "" H 8250 2950 60  0000 C CNN
@@
 $EndComp
 $Comp
-L GND #PWR026
+L GND #PWR025
 U 1 1 54C3C3F0
 P 8000 2950
-F 0 "#PWR026" H 8000 2950 30  0001 C CNN
+F 0 "#PWR025" H 8000 2950 30  0001 C CNN
 F 1 "GND" H 8000 2880 30  0001 C CNN
 F 2 "" H 8000 2950 60  0000 C CNN
@@
 btn3
 $Comp
-L GND #PWR027
+L GND #PWR026
 U 1 1 5589E8F1
 P 6350 4550
-F 0 "#PWR027" H 6350 4550 30  0001 C CNN
+F 0 "#PWR026" H 6350 4550 30  0001 C CNN
 F 1 "GND" H 6350 4480 30  0001 C CNN
 F 2 "" H 6350 4550 60  0000 C CNN
@@
 vdd
 $Comp
-L GND #PWR028
+L GND #PWR027
 U 1 1 55A7B958
 P 6200 6700
-F 0 "#PWR028" H 6200 6700 30  0001 C CNN
+F 0 "#PWR027" H 6200 6700 30  0001 C CNN
 F 1 "GND" H 6200 6630 30  0001 C CNN
 F 2 "" H 6200 6700 60  0000 C CNN
@@
 usb_5v
 $Comp
-L 3310 B1
+L 3310-RESCUE-pitchfork_205_lqfp64 B1
 U 1 1 56C4A80A
 P 8650 4550
@@
 vdd
 $Comp
-L GND #PWR029
+L GND #PWR028
 U 1 1 56C4C8A0
 P 7600 6000
-F 0 "#PWR029" H 7600 6000 30  0001 C CNN
+F 0 "#PWR028" H 7600 6000 30  0001 C CNN
 F 1 "GND" H 7600 5930 30  0001 C CNN
 F 2 "" H 7600 6000 60  0000 C CNN
@@
 vdd
 $Comp
-L GND #PWR030
+L GND #PWR029
 U 1 1 56D33AA1
 P 12300 1600
-F 0 "#PWR030" H 12300 1350 50  0001 C CNN
+F 0 "#PWR029" H 12300 1350 50  0001 C CNN
 F 1 "GND" H 12300 1450 50  0000 C CNN
 F 2 "" H 12300 1600 50  0000 C CNN
@@
 vdd
 $Comp
-L GND #PWR031
+L GND #PWR030
 U 1 1 56D33AB1
 P 15250 1850
-F 0 "#PWR031" H 15250 1600 50  0001 C CNN
+F 0 "#PWR030" H 15250 1600 50  0001 C CNN
 F 1 "GND" H 15250 1700 50  0000 C CNN
 F 2 "" H 15250 1850 50  0000 C CNN
@@
 vdd
 $Comp
-L GND #PWR032
+L GND #PWR031
 U 1 1 56D33AB9
 P 14200 1750
-F 0 "#PWR032" H 14200 1500 50  0001 C CNN
+F 0 "#PWR031" H 14200 1500 50  0001 C CNN
 F 1 "GND" H 14200 1600 50  0000 C CNN
 F 2 "" H 14200 1750 50  0000 C CNN
@@
 $EndComp
 $Comp
-L GND #PWR033
+L GND #PWR032
 U 1 1 56D33ABF
 P 13150 1700
-F 0 "#PWR033" H 13150 1450 50  0001 C CNN
+F 0 "#PWR032" H 13150 1450 50  0001 C CNN
 F 1 "GND" H 13150 1550 50  0000 C CNN
 F 2 "" H 13150 1700 50  0000 C CNN
@@
 $EndComp
 $Comp
-L GND #PWR034
+L GND #PWR033
 U 1 1 56D33ADB
 P 12250 3000
-F 0 "#PWR034" H 12250 2750 50  0001 C CNN
+F 0 "#PWR033" H 12250 2750 50  0001 C CNN
 F 1 "GND" H 12250 2850 50  0000 C CNN
 F 2 "" H 12250 3000 50  0000 C CNN
@@
 $EndComp
 $Comp
-L GND #PWR035
+L GND #PWR034
 U 1 1 56D33AE1
 P 14200 2900
-F 0 "#PWR035" H 14200 2650 50  0001 C CNN
+F 0 "#PWR034" H 14200 2650 50  0001 C CNN
 F 1 "GND" H 14200 2750 50  0000 C CNN
 F 2 "" H 14200 2900 50  0000 C CNN
@@
 $EndComp
 $Comp
-L GND #PWR036
+L GND #PWR035
 U 1 1 56D33AE7
 P 13100 2900
-F 0 "#PWR036" H 13100 2650 50  0001 C CNN
+F 0 "#PWR035" H 13100 2650 50  0001 C CNN
 F 1 "GND" H 13100 2750 50  0000 C CNN
 F 2 "" H 13100 2900 50  0000 C CNN
@@
 $EndComp
 $Comp
-L GND #PWR037
+L GND #PWR036
 U 1 1 56D33B60
 P 14700 1900
-F 0 "#PWR037" H 14700 1650 50  0001 C CNN
+F 0 "#PWR036" H 14700 1650 50  0001 C CNN
 F 1 "GND" H 14700 1750 50  0000 C CNN
 F 2 "" H 14700 1900 50  0000 C CNN
@@
 Text Notes 11650 4050 0    59   ~ 0
 KEYBOARD
+$Comp
+L R_Small R11
+U 1 1 58E8B8A6
+P 8400 3450
+F 0 "R11" H 8430 3470 50  0000 L CNN
+F 1 "10k" H 8430 3410 50  0000 L CNN
+F 2 "opendous:0603_Opendous" H 8400 3450 50  0001 C CNN
+F 3 "" H 8400 3450 50  0000 C CNN
+	1    8400 3450
+	0    1    1    0
+$EndComp
+$Comp
+L GND #PWR037
+U 1 1 58E8BB47
+P 8650 3500
+F 0 "#PWR037" H 8650 3250 50  0001 C CNN
+F 1 "GND" H 8650 3350 50  0000 C CNN
+F 2 "" H 8650 3500 50  0000 C CNN
+F 3 "" H 8650 3500 50  0000 C CNN
+	1    8650 3500
+	1    0    0    -1
+$EndComp
 Wire Wire Line
 	10450 1150 10050 1150
@@
 Wire Wire Line
 	10050 2550 10050 3100
-Connection ~ 8500 3350
 Wire Wire Line
 	4150 3700 4100 3700
@@
 Wire Wire Line
 	8500 2650 8750 2650
-Wire Wire Line
-	9850 3350 9850 3450
-Wire Wire Line
-	8900 3350 9200 3350
-Connection ~ 9850 3350
-Wire Wire Line
-	9850 3350 9600 3350
 Wire Wire Line
 	1900 3950 2150 3950
@@
 	5950 5500 6150 5500
 Wire Wire Line
-	7450 3350 7500 3350
+	7450 3350 7800 3350
 Wire Wire Line
 	6150 6850 5950 6850
@@
 	8000 2750 8750 2750
 Wire Wire Line
-	8500 2550 8500 3350
+	8500 3250 8500 2550
 Connection ~ 8500 2650
 Connection ~ 8500 2750
@@
 	9900 6150 9900 6350
 Connection ~ 7600 5450
-Wire Wire Line
-	8500 3350 8600 3350
 Wire Wire Line
 	10250 3000 10250 2900
@@
 Wire Wire Line
 	3000 700  3500 700
+Wire Wire Line
+	8200 3250 8500 3250
+Wire Wire Line
+	8200 3450 8300 3450
+Wire Wire Line
+	8500 3450 8650 3450
+Wire Wire Line
+	8650 3450 8650 3500
 $EndSCHEMATC
